File: Robot_PCB_(110x55mm).kicad_pcb (KiCad board)
At the start: 2 copper layers, 110 x 55 mm, 20 parts, among them U1 L293, U2 SW_DPDT_XLX, U3 AMS1117-5.0, U5 MFRC522 37.5x25mm

Commit message: update
Parts:
- C5, C6: footprint Capacitor_SMD:C_0603_1608Metric -> Capacitor_SMD:C_0805_2012Metric_Pad1.18x1.45mm_HandSolder

Commit message: Update
Parts:
- added C7: C, Capacitor_SMD:C_0805_2012Metric_Pad1.18x1.45mm_HandSolder, B.Cu at (201.7, 64.6)
- C5, C6: moved to B.Cu
Routing:
- net VCC: track 100.7 -> 114.0 mm
- net +BATT: track 138.1 -> 126.2 mm
- net +5V: track 113.2 -> 118.7 mm, vias 1 -> 0
- net ENC1_B: track 63.5 -> 59.2 mm, vias 1 -> 0
- net MOSI_NRF: track 91.2 -> 86.9 mm, vias 1 -> 0
- net Net-(MOTOR1-Motor_line_+): track 34.5 -> 38.5 mm
- net MISO_NRF: track 84.8 -> 81.1 mm, vias 3 -> 0
- net +3.3V: track 88.0 -> 91.4 mm, vias 1 -> 0
- net SCK_NRF: track 84.8 -> 87.2 mm
- net Net-(MOTOR2-Motor_Line_-): track 102.3 -> 104.5 mm
- net ENC1_A: track 60.6 -> 58.7 mm
- net Net-(MOTOR2-Motor_line_+): track 78.3 -> 79.8 mm
- net CE_NRF: track 82.4 -> 81.7 mm
- net IN4: vias 0 -> 1

Commit message: Update
Parts:
- H1, H2, H3, H4: footprint MountingHole:MountingHole_4mm_Pad -> MountingHole:MountingHole_3.2mm_M3_ISO14580_Pad
- moved NRF24 3.31 mm to (201.7, 58.8)
Routing:
- net +5V: track 118.7 -> 74.2 mm, vias 0 -> 2
- net CE_NRF: track 81.7 -> 121.9 mm, vias 0 -> 1
- net Net-(MOTOR2-Motor_Line_-): track 104.5 -> 82.0 mm
- net IN4: track 40.6 -> 57.8 mm
- net +3V3: track 64.4 -> 80.6 mm, vias 0 -> 1
- net SDA_RFID: track 66.8 -> 82.9 mm
- net VCC: track 114.0 -> 99.6 mm
- net +3.3V: track 91.4 -> 83.1 mm
- net SCK_NRF: track 87.2 -> 80.2 mm, vias 2 -> 0
- net MISO_NRF: track 81.1 -> 88.0 mm, vias 0 -> 1
- net Net-(MOTOR1-Motor_line_+): track 38.5 -> 31.7 mm
- net MOSI_RFID: track 40.4 -> 46.2 mm
- net +BATT: track 126.2 -> 121.9 mm
- net Net-(MOTOR1-Motor_Line_-): track 36.6 -> 39.8 mm
- net MOSI_NRF: track 86.9 -> 83.8 mm
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