File: Robot_PCB_(110x55mm).kicad_pcb (KiCad board)
At the start: 2 copper layers, 110 x 55 mm, 21 parts, among them U1 L293, U2 SW_DPDT_XLX, U3 AMS1117-5.0, U5 MFRC522 37.5x25mm

Commit message: Update
Parts:
- C7: value C -> 100uf
Routing:
- net Net-(MOTOR2-Motor_line_+): track 79.0 -> 78.2 mm
- net ENC2_B: track 10.6 -> 9.97 mm
- net GND: vias 0 -> 10
Other:
- board text added: "JLCJLCJLCJLC"
Changed lines of the file:
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@@
     (property "ki_keywords" "cap capacitor")
     (attr smd)
-    (fp_text reference "C3" (at -2.275 0) (layer "F.SilkS")
+    (fp_text reference "C3" (at -2.275 0) (layer "F.Fab")
         (effects (font (size 1 1) (thickness 0.15)))
     )
@@
     (property "ki_keywords" "mounting hole")
     (attr exclude_from_pos_files)
-    (fp_text reference "H4" (at 0 -3.75) (layer "F.SilkS")
+    (fp_text reference "H4" (at 0 -3.75) (layer "F.SilkS") hide
         (effects (font (size 1 1) (thickness 0.15)))
     )
@@
     (property "ki_keywords" "linear regulator ldo fixed positive")
     (attr smd)
-    (fp_text reference "U3" (at 0.4 2.9) (layer "F.SilkS")
+    (fp_text reference "U3" (at 0.4 2.9) (layer "F.Fab")
         (effects (font (size 1 1) (thickness 0.15)))
     )
@@
     (property "ki_keywords" "ESP32 ")
     (attr through_hole)
-    (fp_text reference "A1" (at 13.253071 1.86 90) (layer "F.SilkS")
+    (fp_text reference "A1" (at 13.253071 1.86 90) (layer "F.Fab")
         (effects (font (size 1 1) (thickness 0.15)))
     )
@@
     (property "ki_description" "Mounting Hole with connection")
     (property "ki_keywords" "mounting hole")
-    (attr exclude_from_pos_files)
-    (fp_text reference "H1" (at 0 -3.75) (layer "F.SilkS")
+    (attr through_hole exclude_from_pos_files)
+    (fp_text reference "H1" (at 0 -3.75) (layer "F.SilkS") hide
         (effects (font (size 1 1) (thickness 0.15)))
     )
@@
     (property "ki_keywords" "cap capacitor")
     (attr smd)
-    (fp_text reference "C2" (at -2.225 -1.43) (layer "F.SilkS")
+    (fp_text reference "C2" (at -2.225 -1.43) (layer "F.Fab")
         (effects (font (size 1 1) (thickness 0.15)))
     )
@@
     (property "ki_keywords" "cap capacitor")
     (attr smd)
-    (fp_text reference "C4" (at -2.275 0) (layer "F.SilkS")
+    (fp_text reference "C4" (at -2.275 0) (layer "F.Fab")
         (effects (font (size 1 1) (thickness 0.15)))
     )
@@
     (property "ki_keywords" "cap capacitor")
     (attr smd)
-    (fp_text reference "C1" (at 2.225 -1.5) (layer "F.SilkS")
+    (fp_text reference "C1" (at 2.225 -1.5) (layer "F.Fab")
         (effects (font (size 1 1) (thickness 0.15)))
     )
@@
     (property "ki_description" "Mounting Hole with connection")
     (property "ki_keywords" "mounting hole")
-    (attr exclude_from_pos_files)
-    (fp_text reference "H2" (at 0 -3.75) (layer "F.SilkS")
+    (attr through_hole exclude_from_pos_files)
+    (fp_text reference "H2" (at 0 -3.75) (layer "F.SilkS") hide
         (effects (font (size 1 1) (thickness 0.15)))
     )
@@
     (property "ki_keywords" "mounting hole")
     (attr exclude_from_pos_files)
-    (fp_text reference "H3" (at 0 -3.75) (layer "F.SilkS")
+    (fp_text reference "H3" (at 0 -3.75) (layer "F.SilkS") hide
         (effects (font (size 1 1) (thickness 0.15)))
     )
@@
       (net 18 "+BATT") (pintype "passive"))
     (pad "2" thru_hole oval locked (at 2.5 0 180) (size 1.7 2) (drill 1) (layers "*.Cu" "*.Mask")
-      (net 41 "GND") (pintype "passive"))
+      (net 41 "GND") (pintype "passive") (zone_connect 1))
     (model "${KICAD6_3DMODEL_DIR}/Connector_JST.3dshapes/JST_EH_B2B-EH-A_1x02_P2.50mm_Vertical.wrl"
       (offset (xyz 0 0 0))
@@
     (property "ki_description" "Quadruple Half-H Drivers")
     (property "ki_keywords" "Half-H Driver Motor")
-    (fp_text reference "U1" (at 0.05 -2.4 90) (layer "F.SilkS")
+    (zone_connect 1)
+    (fp_text reference "U1" (at 0.05 -2.4 90) (layer "F.Fab")
         (effects (font (size 1 1) (thickness 0.15)))
     )
@@
     (property "ki_keywords" "cap capacitor")
     (attr smd)
-    (fp_text reference "C6" (at 0 1.68) (layer "B.SilkS")
+    (fp_text reference "C6" (at 0 1.68) (layer "B.Fab")
         (effects (font (size 1 1) (thickness 0.15)) (justify mirror))
     )
@@
     (property "ki_keywords" "cap capacitor")
     (attr smd)
-    (fp_text reference "C5" (at 0 1.68) (layer "B.SilkS")
+    (fp_text reference "C5" (at 0 1.68) (layer "B.Fab")
         (effects (font (size 1 1) (thickness 0.15)) (justify mirror))
     )
@@
     (property "ki_keywords" "cap capacitor")
     (attr smd)
-    (fp_text reference "C7" (at 0 1.68 90) (layer "B.SilkS")
+    (fp_text reference "C7" (at 0 1.73 180) (layer "F.Fab")
         (effects (font (size 1 1) (thickness 0.15)) (justify mirror))
     )
-    (fp_text value "C" (at 0 -1.68 90) (layer "B.Fab")
+    (fp_text value "100uf" (at 0 -1.68 90) (layer "B.Fab")
         (effects (font (size 1 1) (thickness 0.15)) (justify mirror))
     )
@@
   (gr_arc (start 105 100) (mid 101.464466 98.535534) (end 100 95)
     (stroke (width 0.1) (type default)) (layer "Edge.Cuts"))
+  (gr_text "JLCJLCJLCJLC" (at 113 72.5) (layer "F.SilkS")
+    (effects (font (size 1 1) (thickness 0.17) bold) (justify left bottom))
+  )
   (dimension (type aligned) (layer "Cmts.User")
     (pts (xy 182 75.8) (xy 188.5 75.8))
@@
   (segment (start 137.43 60.12) (end 137.12 60.12) (width 0.3) (layer "B.Cu") (net 16))
   (segment (start 137.12 60.12) (end 130 53) (width 0.3) (layer "B.Cu") (net 16))
-  (segment (start 128 54.2809) (end 129.051 54.2809) (width 0.3) (layer "B.Cu") (net 17))
-  (segment (start 129.051 54.2809) (end 134.89 60.12) (width 0.3) (layer "B.Cu") (net 17))
-  (segment (start 128 53) (end 128 54.2809) (width 0.3) (layer "B.Cu") (net 17))
+  (segment (start 128 53) (end 128 53.23) (width 0.3) (layer "B.Cu") (net 17))
+  (segment (start 128 53.23) (end 134.89 60.12) (width 0.3) (layer "B.Cu") (net 17))
   (segment (start 138.065 78.724) (end 146.473 78.724) (width 1) (layer "F.Cu") (net 18))
   (segment (start 123.81 76.54) (end 125.512 76.54) (width 1) (layer "F.Cu") (net 18))
@@
   (segment (start 152.45 98.37) (end 147.74 98.37) (width 0.3) (layer "B.Cu") (net 20))
   (segment (start 134.772 72.8275) (end 133.555 72.8275) (width 0.3) (layer "F.Cu") (net 21))
+  (segment (start 137.1118 73.4382) (end 136.95 73.6) (width 0.3) (layer "F.Cu") (net 21))
   (segment (start 136.95 73.6) (end 135.544 73.6) (width 0.3) (layer "F.Cu") (net 21))
   (segment (start 146.227 75.4239) (end 146.227 75.7559) (width 0.3) (layer "F.Cu") (net 21))
   (segment (start 135.544 73.6) (end 134.772 72.8275) (width 0.3) (layer "F.Cu") (net 21))
+  (segment (start 138.356 73.4382) (end 137.1118 73.4382) (width 0.3) (layer "F.Cu") (net 21))
   (segment (start 143.25 73.6) (end 143.25 72.447) (width 0.3) (layer "F.Cu") (net 21))
-  (segment (start 136.95 73.6) (end 138.356 73.6) (width 0.3) (layer "F.Cu") (net 21))
-  (segment (start 143.25 71.2941) (end 140.5 71.2941) (width 0.3) (layer "F.Cu") (net 21))
-  (segment (start 143.25 72.447) (end 143.25 71.2941) (width 0.3) (layer "F.Cu") (net 21))
   (segment (start 138.356 73.4382) (end 140.5 71.2941) (width 0.3) (layer "F.Cu") (net 21))
-  (segment (start 138.356 73.6) (end 138.356 73.4382) (width 0.3) (layer "F.Cu") (net 21))
+  (segment (start 140.5 71.2941) (end 140.9441 71.2941) (width 0.3) (layer "F.Cu") (net 21))
+  (segment (start 140.9441 71.2941) (end 143.25 73.6) (width 0.3) (layer "F.Cu") (net 21))
   (segment (start 143.25 72.447) (end 146.227 75.4239) (width 0.3) (layer "F.Cu") (net 21))
   (segment (start 140.5 69) (end 140.5 67.5) (width 0.3) (layer "F.Cu") (net 21))
@@
   (segment (start 179.962 55.89) (end 179.9623 55.8898) (width 0.85) (layer "B.Cu") (net 39))
   (segment (start 179.9623 55.8898) (end 180 55.8525) (width 0.85) (layer "B.Cu") (net 39))
-  (segment (start 118.73 76.54) (end 118.73 78.5169) (width 0.85) (layer "B.Cu") (net 39))
+  (segment (start 120.02 78.5169) (end 131.393 78.5169) (width 0.85) (layer "B.Cu") (net 39))
   (segment (start 131.393 78.5169) (end 158.512 51.3981) (width 0.85) (layer "B.Cu") (net 39))
+  (segment (start 118.73 77.2269) (end 120.02 78.5169) (width 0.85) (layer "B.Cu") (net 39))
   (segment (start 180 55.8525) (end 180 53) (width 0.85) (layer "B.Cu") (net 39))
   (segment (start 180 51.3981) (end 180 53) (width 0.85) (layer "B.Cu") (net 39))
   (segment (start 158.512 51.3981) (end 180 51.3981) (width 0.85) (layer "B.Cu") (net 39))
-  (segment (start 118.73 78.5169) (end 131.393 78.5169) (width 0.85) (layer "B.Cu") (net 39))
+  (segment (start 118.73 76.54) (end 118.73 77.2269) (width 0.85) (layer "B.Cu") (net 39))
   (segment (start 179.9625 55.89) (end 179.9623 55.8898) (width 0.85) (layer "B.Cu") (net 39))
   (segment (start 177.8875 55.89) (end 177.888 55.89) (width 0.85) (layer "B.Cu") (net 40))
@@
   (segment (start 112.286 79.6929) (end 131.938 79.6929) (width 0.85) (layer "B.Cu") (net 40))
   (segment (start 111.11 76.54) (end 111.11 78.5169) (width 0.85) (layer "B.Cu") (net 40))
+  (via (at 160 66) (size 0.8) (drill 0.4) (layers "F.Cu" "B.Cu") (free) (net 41))
+  (via (at 165 90) (size 0.8) (drill 0.4) (layers "F.Cu" "B.Cu") (free) (net 41))
+  (via (at 142 53) (size 0.8) (drill 0.4) (layers "F.Cu" "B.Cu") (free) (net 41))
+  (via (at 146 90) (size 0.8) (drill 0.4) (layers "F.Cu" "B.Cu") (free) (net 41))
+  (via (at 168 49) (size 0.8) (drill 0.4) (layers "F.Cu" "B.Cu") (free) (net 41))
+  (via (at 180 66) (size 0.8) (drill 0.4) (layers "F.Cu" "B.Cu") (free) (net 41))
+  (via (at 147 58) (size 0.8) (drill 0.4) (layers "F.Cu" "B.Cu") (free) (net 41))
+  (via (at 136 90) (size 0.8) (drill 0.4) (layers "F.Cu" "B.Cu") (free) (net 41))
+  (via (at 153 90) (size 0.8) (drill 0.4) (layers "F.Cu" "B.Cu") (free) (net 41))
+  (via (at 178 66) (size 0.8) (drill 0.4) (layers "F.Cu" "B.Cu") (free) (net 41))
   (segment (start 139.81 76.9578) (end 181.25 76.9578) (width 1) (layer "F.Cu") (net 42))
   (segment (start 134.928 75.9) (end 136.95 75.9) (width 1) (layer "F.Cu") (net 42))
@@
     (connect_pads (clearance 0.3))
     (min_thickness 0.3) (filled_areas_thickness no)
-    (fill yes (thermal_gap 0.2) (thermal_bridge_width 0.8) (island_removal_mode 1) (island_area_min 10))
+    (fill yes (thermal_gap 0.4) (thermal_bridge_width 0.7) (island_removal_mode 1) (island_area_min 10))
     (polygon
       (pts

Commit message: Update
Parts:
- H1, H2, H3, H4: footprint MountingHole:MountingHole_3.2mm_M3_ISO14580_Pad -> MountingHole:MountingHole_3.2mm_M3_DIN965_Pad
Routing:
- net Net-(MOTOR2-Motor_line_+): track 78.2 -> 128.2 mm
- net CE_NRF: track 121.9 -> 81.1 mm
- net MOSI_NRF: track 83.8 -> 104.4 mm
- net Net-(MOTOR2-Motor_Line_-): track 82.0 -> 101.7 mm
- net IN4: track 57.8 -> 40.1 mm
- net +3V3: track 80.6 -> 63.3 mm
- net SDA_RFID: track 82.9 -> 65.9 mm
- net +BATT: track 121.9 -> 138.2 mm
- net VCC: track 99.6 -> 110.9 mm
- net MISO_NRF: track 88.0 -> 78.8 mm, vias 1 -> 0
- net +3.3V: track 83.1 -> 88.9 mm
- net MOSI_RFID: track 46.2 -> 40.4 mm
- net +5V: track 73.9 -> 79.6 mm, vias 2 -> 1
- net ENC1_A: track 56.6 -> 61.3 mm, vias 0 -> 1
- net CSN_NRF: track 94.6 -> 99.0 mm
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
Commit message: Update
Parts:
- removed C3: 10uf, Capacitor_SMD:C_0603_1608Metric
- removed C4: 100uf, Capacitor_SMD:C_0603_1608Metric
- C1: value 10uf -> 100nF; footprint Capacitor_SMD:C_0603_1608Metric -> Capacitor_SMD:C_0805_2012Metric_Pad1.18x1.45mm_HandSolder; moved to B.Cu
- C2: value 100uf -> 220uF_10V; footprint Capacitor_SMD:C_0603_1608Metric -> Capacitor_THT:CP_Radial_D6.3mm_P2.50mm
- C5, C6: value C -> 100nF
- U3: moved to B.Cu
- moved C1 43.0 mm to (172.8, 81.5), turned to 90 degrees
- moved U3 28.6 mm to (166.8, 84.0), turned to -90 degrees
- moved C2 21.1 mm to (143.5, 52.5)
Connections:
- C2 pad 1: VCC -> +5V
Routing:
- net Net-(MOTOR2-Motor_line_+): track 128.2 -> 75.4 mm
- net VCC: track 110.9 -> 149.5 mm
- net +BATT: track 138.2 -> 108.2 mm
- net +5V: track 79.6 -> 109.5 mm
- net Net-(MOTOR2-Motor_Line_-): track 101.7 -> 80.8 mm
- net MISO_NRF: track 78.8 -> 88.6 mm
- net CE_NRF: track 81.1 -> 88.2 mm
- net MOSI_NRF: track 104.4 -> 97.3 mm
- net SCK_NRF: track 80.6 -> 87.2 mm
- net +3.3V: track 88.9 -> 83.5 mm
- net IN4: track 40.1 -> 45.4 mm
- net Net-(MOTOR1-Motor_line_+): track 32.2 -> 37.4 mm
- net Net-(MOTOR1-Motor_Line_-): track 38.1 -> 35.4 mm
- net ENC1_B: track 60.9 -> 58.7 mm
- net CSN_NRF: track 99.0 -> 97.2 mm, vias 1 -> 0
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
Commit message: Update
Parts:
- moved C7 0.14 mm to (201.8, 64.8)
Routing:
- net VCC: track 149.5 -> 153.8 mm
- net +3.3V: track 83.5 -> 84.9 mm
- net Net-(MOTOR1-Motor_Line_-): track 35.4 -> 36.7 mm
- net MISO_NRF: track 88.6 -> 89.9 mm
- net Net-(MOTOR1-Motor_line_+): track 37.4 -> 38.5 mm
- net +3V3: track 63.3 -> 64.1 mm

Commit message: Update
Routing:
- net Net-(MOTOR2-Motor_Line_-): track 80.8 -> 81.3 mm

Commit message: Update
Routing:
- net Net-(MOTOR1-Motor_line_+): track 38.5 -> 41.5 mm
- net Net-(MOTOR1-Motor_Line_-): track 36.7 -> 38.9 mm
- net ENC1_B: track 58.7 -> 59.3 mm

Commit message: Update
Parts:
- renumbered MOTOR2 to MOTOR1, MOTOR1 to MOTOR2
Routing:
- net CE_NRF: track 88.2 -> 88.8 mm
- net GND: vias 28 -> 23

Commit message: update
Parts:
- moved BAT1 2.50 mm to (153.8, 48.8), turned to 0 degrees
Connections:
- BAT1 pad 1: +BATT -> GND
- BAT1 pad 2: GND -> +BATT
Other:
- board text added: "+"
Changed lines of the file:
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@@
   )
   (footprint "Connector_JST:JST_EH_B2B-EH-A_1x02_P2.50mm_Vertical" locked (layer "F.Cu")
-    (at 156.25 48.8 180)
+    (at 153.75 48.75)
     (descr "JST EH series connector, B2B-EH-A (http://www.jst-mfg.com/product/pdf/eng/eEH.pdf), generated with kicad-footprint-generator")
     (tags "connector JST EH vertical")
@@
     (property "ki_keywords" "JST 2")
     (attr through_hole)
-    (fp_text reference "BAT1" (at 1.25 -2.8) (layer "F.SilkS")
+    (fp_text reference "BAT1" (at 1.5 3.5) (layer "F.SilkS") hide
         (effects (font (size 1 1) (thickness 0.15)))
     )
-    (fp_text value "JST_02" (at 1.25 3.4) (layer "F.Fab")
+    (fp_text value "JST_02" (at -3.5 0) (layer "F.Fab")
         (effects (font (size 1 1) (thickness 0.15)))
     )
@@
     (fp_line (start 5 2.2) (end 5 -1.6)
       (stroke (width 0.1) (type solid)) (layer "F.Fab"))
-    (pad "1" thru_hole roundrect locked (at 0 0 180) (size 1.7 2) (drill 1) (layers "*.Cu" "*.Mask") (roundrect_rratio 0.147059)
+    (pad "1" thru_hole roundrect locked (at 0 0) (size 1.7 2) (drill 1) (layers "*.Cu" "*.Mask") (roundrect_rratio 0.147059)
+      (net 40 "GND") (pintype "passive"))
+    (pad "2" thru_hole oval locked (at 2.5 0) (size 1.7 2) (drill 1) (layers "*.Cu" "*.Mask")
       (net 17 "+BATT") (pintype "passive"))
-    (pad "2" thru_hole oval locked (at 2.5 0 180) (size 1.7 2) (drill 1) (layers "*.Cu" "*.Mask")
-      (net 40 "GND") (pintype "passive"))
     (model "${KICAD6_3DMODEL_DIR}/Connector_JST.3dshapes/JST_EH_B2B-EH-A_1x02_P2.50mm_Vertical.wrl"
       (offset (xyz 0 0 0))
@@
   (gr_arc (start 105 100) (mid 101.464466 98.535534) (end 100 95)
     (stroke (width 0.1) (type default)) (layer "Edge.Cuts"))
+  (gr_text "+" (at 159.25 49.25) (layer "F.SilkS")
+    (effects (font (size 1 1) (thickness 0.15)) (justify left bottom))
+  )
   (gr_text "JLCJLCJLCJLC" (at 109.5 65.5) (layer "F.SilkS")
     (effects (font (size 1 1) (thickness 0.17) bold) (justify left bottom))
@@
   (segment (start 128 53.23) (end 134.89 60.12) (width 0.4) (layer "F.Cu") (net 16))
   (segment (start 128 53) (end 128 53.23) (width 0.4) (layer "F.Cu") (net 16))
-  (segment (start 156.025 62.8) (end 156.025 49.025) (width 1) (layer "B.Cu") (net 17))
+  (segment (start 156.25 62.575) (end 156.25 48.8) (width 1) (layer "B.Cu") (net 17))
+  (segment (start 156.25 62.575) (end 158.175 64.5) (width 1) (layer "B.Cu") (net 17))
+  (segment (start 158.175 64.5) (end 171 64.5) (width 1) (layer "B.Cu") (net 17))
+  (segment (start 171 64.5) (end 195.5 89) (width 1) (layer "B.Cu") (net 17))
+  (segment (start 153 65.825) (end 156.25 62.575) (width 1) (layer "B.Cu") (net 17))
   (segment (start 195.5 92.1019) (end 194.302 93.3) (width 1) (layer "B.Cu") (net 17))
+  (segment (start 134.325 65.825) (end 153 65.825) (width 1) (layer "B.Cu") (net 17))
   (segment (start 194.302 93.3) (end 193.05 93.3) (width 1) (layer "B.Cu") (net 17))
-  (segment (start 195.5 89) (end 195.5 92.1019) (width 1) (layer "B.Cu") (net 17))
-  (segment (start 156.025 62.8) (end 157.725 64.5) (width 1) (layer "B.Cu") (net 17))
-  (segment (start 171 64.5) (end 195.5 89) (width 1) (layer "B.Cu") (net 17))
-  (segment (start 157.725 64.5) (end 171 64.5) (width 1) (layer "B.Cu") (net 17))
-  (segment (start 156.025 49.025) (end 156.25 48.8) (width 1) (layer "B.Cu") (net 17))
-  (segment (start 134.325 65.825) (end 153 65.825) (width 1) (layer "B.Cu") (net 17))
-  (segment (start 153 65.825) (end 156.025 62.8) (width 1) (layer "B.Cu") (net 17))
   (segment (start 123.81 76.54) (end 123.81 76.34) (width 1) (layer "B.Cu") (net 17))
   (segment (start 123.81 76.34) (end 134.325 65.825) (width 1) (layer "B.Cu") (net 17))
+  (segment (start 195.5 89) (end 195.5 92.1019) (width 1) (layer "B.Cu") (net 17))
   (segment (start 156.26 97.1) (end 154.283 99.0769) (width 0.4) (layer "B.Cu") (net 18))
   (segment (start 154.283 99.0769) (end 138.287 99.0769) (width 0.4) (layer "B.Cu") (net 18))
