File: Robot_PCB_(110x55mm).kicad_pcb (KiCad board)
At the start: 2 copper layers, 110 x 55 mm, 19 parts, among them U1 L293, U2 SW_DPDT_XLX, U3 AMS1117-5.0, U5 MFRC522 37.5x25mm

Commit message: Update
Connections:
- net ENC1_A renamed M1_S1
- net ENC1_B renamed M1_S2
- net ENC2_A renamed M2_S1
- net ENC2_B renamed M2_S2
- C5 pad 1: Net-(MOTOR2-Motor_Line_-) -> Net-(U1-4Y)
- C5 pad 2: Net-(MOTOR2-Motor_line_+) -> Net-(U1-3Y)
- C6 pad 1: Net-(MOTOR1-Motor_Line_-) -> Net-(U1-2Y)
- C6 pad 2: Net-(MOTOR1-Motor_line_+) -> Net-(U1-1Y)
- MOTOR1 pad 5: Net-(MOTOR1-Motor_line_+) -> Net-(U1-1Y)
- MOTOR1 pad 6: Net-(MOTOR1-Motor_Line_-) -> Net-(U1-2Y)
- MOTOR2 pad 5: Net-(MOTOR2-Motor_line_+) -> Net-(U1-3Y)
- MOTOR2 pad 6: Net-(MOTOR2-Motor_Line_-) -> Net-(U1-4Y)
- U1 pad 11: Net-(MOTOR2-Motor_Line_-) -> Net-(U1-3Y)
- U1 pad 14: Net-(MOTOR2-Motor_line_+) -> Net-(U1-4Y)
- U1 pad 3: Net-(MOTOR1-Motor_Line_-) -> Net-(U1-1Y)
- U1 pad 6: Net-(MOTOR1-Motor_line_+) -> Net-(U1-2Y)
Routing:
- net Net-(U1-1Y): track 0.00 -> 81.5 mm
- net Net-(MOTOR1-Motor_Line_-): track 81.3 -> 0.00 mm
- net Net-(MOTOR1-Motor_line_+): track 75.4 -> 0.00 mm
- net Net-(U1-2Y): track 0.00 -> 72.0 mm, vias 0 -> 1
- net Net-(U1-3Y): track 0.00 -> 50.5 mm
- net Net-(MOTOR2-Motor_line_+): track 41.5 -> 0.00 mm
- net Net-(MOTOR2-Motor_Line_-): track 38.9 -> 0.00 mm
- net Net-(U1-4Y): track 0.00 -> 29.2 mm

Commit message: Update 17:35
Parts:
- moved BAT1 0.25 mm to (153.5, 48.8)
Connections:
- C5 pad 1: Net-(U1-4Y) -> /M2-
- C5 pad 2: Net-(U1-3Y) -> /M2+
- C6 pad 1: Net-(U1-2Y) -> /M1-
- C6 pad 2: Net-(U1-1Y) -> /M1+
- C7 pad 1: +3.3V -> +3V3
- MOTOR1 pad 4: +3.3V -> +3V3
- MOTOR1 pad 5: Net-(U1-1Y) -> /M1+
- MOTOR1 pad 6: Net-(U1-2Y) -> /M1-
- MOTOR2 pad 4: +3.3V -> +3V3
- MOTOR2 pad 5: Net-(U1-3Y) -> /M2+
- MOTOR2 pad 6: Net-(U1-4Y) -> /M2-
- NRF24 pad 2: +3.3V -> +3V3
- U1 pad 11: Net-(U1-3Y) -> /M2-
- U1 pad 14: Net-(U1-4Y) -> /M2+
- U1 pad 3: Net-(U1-1Y) -> /M1-
- U1 pad 6: Net-(U1-2Y) -> /M1+
Routing:
- net +3V3: track 64.1 -> 160.9 mm, vias 0 -> 1
- net +3.3V: track 84.6 -> 0.00 mm
- net Net-(U1-1Y): track 81.5 -> 0.00 mm
- net /M1-: track 0.00 -> 81.1 mm
- net /M1+: track 0.00 -> 75.4 mm
- net Net-(U1-2Y): track 72.0 -> 0.00 mm, vias 1 -> 0
- net Net-(U1-3Y): track 50.5 -> 0.00 mm
- net /M2+: track 0.00 -> 41.5 mm
- net /M2-: track 0.00 -> 38.9 mm
- net Net-(U1-4Y): track 29.2 -> 0.00 mm

Commit message: Update 11:14 - 21/10/23
Connections:
- U1 pad 8: +BATT -> VCC
Routing:
- net +3V3: track 160.9 -> 231.6 mm, vias 1 -> 0
- net +BATT: track 108.7 -> 69.6 mm
- net VCC: track 153.8 -> 178.8 mm
- net GND: vias 23 -> 25

Commit message: Update
Parts:
- moved C2 3.95 mm to (147.2, 53.8), turned to 180 degrees
- moved C5 0.19 mm to (122.9, 55.8)
- moved C6 0.14 mm to (178.9, 55.8)
Routing:
- net +5V: track 109.8 -> 117.6 mm
- net +3V3: track 231.6 -> 232.4 mm

Commit message: Update
Parts:
- added BZ1: Buzzer, Buzzer_Beeper:Buzzer_12x9.5RM7.6, F.Cu at (129.0, 93.5)
- added Q1: J3, Package_TO_SOT_SMD:SOT-23_Handsoldering, B.Cu at (145.2, 93.0)
- added R1: 1000, Resistor_SMD:R_0805_2012Metric_Pad1.20x1.40mm_HandSolder, B.Cu at (139.8, 92.0)
- added R2: 330, Resistor_SMD:R_0805_2012Metric_Pad1.20x1.40mm_HandSolder, B.Cu at (156.3, 91.1)
- added R3: 680, Resistor_SMD:R_0805_2012Metric_Pad1.20x1.40mm_HandSolder, B.Cu at (160.0, 91.1)
- SW1: renamed from U2; value SW_DPDT_XLX -> Switch; footprint GERE_footprints:SW_DPDT_XLX -> GERE_footprints:Push Button Switch 7mm
- moved SW1 3.54 mm to (193.5, 95.8), turned to 0 degrees
Connections:
- A1 pad 14: unconnected-(A1-D22/SCL-Pad14) -> BUZZER
- HC-SR04 pad 2: Echo -> Net-(HC-SR04-Pad2)
Routing:
- net Net-(BZ1--): track 0.00 -> 22.7 mm, vias 0 -> 1
- net Echo: track 38.0 -> 57.6 mm
- net +5V: track 117.6 -> 125.3 mm
- net BUZZER: track 0.00 -> 6.99 mm
- net Net-(HC-SR04-Pad2): track 0.00 -> 5.13 mm
- net Net-(Q1-B): track 0.00 -> 5.12 mm
- net Trig: track 24.7 -> 29.3 mm
- net VCC: track 178.8 -> 179.4 mm
- net GND: vias 25 -> 26

Commit message: Update
Parts:
- removed HC-SR04: PINHD_1x4_Female, Connector_PinSocket_2.54mm:PinSocket_1x04_P2.54mm_Vertical
- added J1: HC-SR04, GERE_footprints:HC-SR04, F.Cu at (158.8, 97.0)
- renumbered C2 to C1, C1 to C2, C5 to C3, C6 to C4, C7 to C5, U3 to U2
Routing:
- net +5V: track 125.3 -> 134.5 mm
- net Net-(J1-Trig): track 5.13 -> 9.75 mm
- net Trig: track 29.3 -> 30.3 mm
- net GND: vias 26 -> 34

Commit message: Update
Parts:
- removed BZ1: Buzzer, Buzzer_Beeper:Buzzer_12x9.5RM7.6
- removed Q1: J3, Package_TO_SOT_SMD:SOT-23_Handsoldering
- added D1: LED, LED_THT:LED_D3.0mm_Clear, F.Cu at (118.8, 95.2)
- added G***: LOGO, GERE_footprints:info2, F.Cu at (116.0, 95.2)
- R1: value 1000 -> ~
- moved R1 2.89 mm to (142.5, 91.1)
Connections:
- net BUZZER renamed LED
Routing:
- net Net-(BZ1--): track 22.7 -> 0.00 mm, vias 1 -> 0
- net Net-(D1-A): track 5.12 -> 22.5 mm, vias 0 -> 1
- net +5V: track 134.5 -> 127.0 mm
- net LED: track 6.99 -> 4.95 mm
