File: Robot_PCB_(110x55mm).kicad_sch (KiCad schematic)
At the start: 20 parts, among them U1 L293, U2 SW_DPDT_XLX, U3 AMS1117-5.0, U5 MFRC522 37.5x25mm

Commit message: update
Parts:
- C5, C6: footprint Capacitor_SMD:C_0603_1608Metric -> Capacitor_SMD:C_0805_2012Metric_Pad1.18x1.45mm_HandSolder
Other:
- moved on the sheet: C1, C2, C3, C4, U3

Commit message: Update
Parts:
- added C7: C, Capacitor_SMD:C_0805_2012Metric_Pad1.18x1.45mm_HandSolder, symbol Device:C
Connections:
- net +3.3V: now also C7.1
- net GND: now also C7.2
Changed lines of the file:
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@@
   (junction (at 175.895 32.512) (diameter 0) (color 0 0 0 0)
   )
+  (junction (at 235.712 137.16) (diameter 0) (color 0 0 0 0)
+  )
   (junction (at 201.295 32.512) (diameter 0) (color 0 0 0 0)
   )
@@
     (stroke (width 0) (type default))
   )
+  (wire (pts (xy 235.712 133.604) (xy 235.712 137.16))
+    (stroke (width 0) (type default))
+  )
+  (wire (pts (xy 245.11 137.414) (xy 246.126 137.414))
+    (stroke (width 0) (type default))
+  )
   (wire (pts (xy 51.308 98.298) (xy 43.815 98.298))
     (stroke (width 0) (type default))
@@
     (stroke (width 0) (type default))
   )
+  (wire (pts (xy 237.49 137.414) (xy 235.966 137.414))
+    (stroke (width 0) (type default))
+  )
   (wire (pts (xy 170.18 114.935) (xy 172.72 114.935))
     (stroke (width 0) (type default))
@@
     (stroke (width 0) (type default))
   )
-  (wire (pts (xy 235.839 139.7) (xy 235.839 138.176))
+  (wire (pts (xy 235.712 139.7) (xy 235.712 137.16))
     (stroke (width 0) (type default))
   )
@@
     (stroke (width 0) (type default))
   )
-  (wire (pts (xy 234.315 139.7) (xy 235.839 139.7))
+  (wire (pts (xy 234.315 139.7) (xy 235.712 139.7))
     (stroke (width 0) (type default))
   )
@@
     (stroke (width 0) (type default))
   )
+  (wire (pts (xy 235.966 137.414) (xy 235.966 137.16))
+    (stroke (width 0) (type default))
+  )
   (wire (pts (xy 201.295 32.512) (xy 201.295 37.592))
     (stroke (width 0) (type default))
@@
   )
   (wire (pts (xy 181.61 32.512) (xy 184.15 32.512))
+    (stroke (width 0) (type default))
+  )
+  (wire (pts (xy 235.966 137.16) (xy 235.712 137.16))
     (stroke (width 0) (type default))
   )
@@
     (fill (type none))
   )
-  (rectangle (start 197.358 128.778) (end 254 154.178)
+  (rectangle (start 197.358 126.746) (end 254 154.178)
     (stroke (width 0) (type dash))
     (fill (type none))
@@
     (fill (type none))
   )
-  (text "NRF24" (at 204.343 132.588 0)
+  (text "NRF24" (at 199.898 130.048 0)
     (effects (font (size 1.27 1.27)) (justify left bottom))
   )
@@
         (path "/5740c1d8-40a5-48a4-b0ff-1fed8540b5f6"
           (reference "#PWR05") (unit 1)
+        )
+      )
+    )
+  )
+  (symbol (lib_id "Device:C") (at 241.3 137.414 90) (unit 1)
+    (in_bom yes) (on_board yes) (dnp no)
+    (property "Reference" "C7" (at 244.602 131.826 90)
+      (effects (font (size 1.27 1.27)))
+    )
+    (property "Value" "C" (at 241.3 132.334 90)
+      (effects (font (size 1.27 1.27)))
+    )
+    (property "Footprint" "Capacitor_SMD:C_0805_2012Metric_Pad1.18x1.45mm_HandSolder" (at 245.11 136.4488 0)
+      (effects (font (size 1.27 1.27)) hide)
+    )
+    (property "Datasheet" "~" (at 241.3 137.414 0)
+      (effects (font (size 1.27 1.27)) hide)
+    )
+    (pin "1")
+    (pin "2")
+    (instances
+      (project "Robot_PCB_(110x55mm)"
+        (path "/5740c1d8-40a5-48a4-b0ff-1fed8540b5f6"
+          (reference "C7") (unit 1)
         )
       )
@@
     )
   )
-  (symbol (lib_id "power:+3.3V") (at 235.839 138.176 0) (unit 1)
-    (in_bom yes) (on_board yes) (dnp no) (fields_autoplaced)
-    (property "Reference" "#PWR027" (at 235.839 141.986 0)
-      (effects (font (size 1.27 1.27)) hide)
-    )
-    (property "Value" "+3.3V" (at 235.839 133.858 0)
-      (effects (font (size 1.27 1.27)))
-    )
-    (property "Footprint" "" (at 235.839 138.176 0)
-      (effects (font (size 1.27 1.27)) hide)
-    )
-    (property "Datasheet" "" (at 235.839 138.176 0)
+  (symbol (lib_id "power:+3.3V") (at 235.712 133.604 0) (unit 1)
+    (in_bom yes) (on_board yes) (dnp no) (fields_autoplaced)
+    (property "Reference" "#PWR027" (at 235.712 137.414 0)
+      (effects (font (size 1.27 1.27)) hide)
+    )
+    (property "Value" "+3.3V" (at 235.712 129.286 0)
+      (effects (font (size 1.27 1.27)))
+    )
+    (property "Footprint" "" (at 235.712 133.604 0)
+      (effects (font (size 1.27 1.27)) hide)
+    )
+    (property "Datasheet" "" (at 235.712 133.604 0)
       (effects (font (size 1.27 1.27)) hide)
     )
@@
         )
       )
+    )
+  )
+  (symbol (lib_id "power:GND") (at 246.126 137.414 90) (unit 1)
+    (in_bom yes) (on_board yes) (dnp no) (fields_autoplaced)
+    (property "Reference" "#PWR029" (at 252.476 137.414 0)
+      (effects (font (size 1.27 1.27)) hide)
+    )
+    (property "Value" "GND" (at 250.19 137.414 90)
+      (effects (font (size 1.27 1.27)) (justify right))
+    )
+    (property "Footprint" "" (at 246.126 137.414 0)
+      (effects (font (size 1.27 1.27)) hide)
+    )
+    (property "Datasheet" "" (at 246.126 137.414 0)
+      (effects (font (size 1.27 1.27)) hide)
+    )
+    (pin "1")
+    (instances
+      (project "Robot_PCB_(110x55mm)"
+        (path "/5740c1d8-40a5-48a4-b0ff-1fed8540b5f6"
+          (reference "#PWR029") (unit 1)
+        )
+      )

Commit message: Update
Parts:
- H1, H2, H3, H4: footprint MountingHole:MountingHole_4mm_Pad -> MountingHole:MountingHole_3.2mm_M3_ISO14580_Pad
Changed lines of the file:
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@@
       (effects (font (size 1.27 1.27)) (justify left))
     )
-    (property "Footprint" "MountingHole:MountingHole_4mm_Pad" (at 16.764 17.272 0)
+    (property "Footprint" "MountingHole:MountingHole_3.2mm_M3_ISO14580_Pad" (at 16.764 17.272 0)
       (effects (font (size 1.27 1.27)) hide)
     )
@@
       (effects (font (size 1.27 1.27)) (justify left))
     )
-    (property "Footprint" "MountingHole:MountingHole_4mm_Pad" (at 24.638 24.892 0)
+    (property "Footprint" "MountingHole:MountingHole_3.2mm_M3_ISO14580_Pad" (at 24.638 24.892 0)
       (effects (font (size 1.27 1.27)) hide)
     )
@@
       (effects (font (size 1.27 1.27)) (justify left))
     )
-    (property "Footprint" "MountingHole:MountingHole_4mm_Pad" (at 16.256 24.892 0)
+    (property "Footprint" "MountingHole:MountingHole_3.2mm_M3_ISO14580_Pad" (at 16.256 24.892 0)
       (effects (font (size 1.27 1.27)) hide)
     )
@@
       (effects (font (size 1.27 1.27)) (justify left))
     )
-    (property "Footprint" "MountingHole:MountingHole_4mm_Pad" (at 24.638 17.272 0)
-      (effects (font (size 1.27 1.27)) hide)
-    )
+    (property "Footprint" "MountingHole:MountingHole_3.2mm_M3_ISO14580_Pad" (at 24.638 17.272 0)
+      (effects (font (size 1.27 1.27)) hide)
+    )

Commit message: Update
Parts:
- C7: value C -> 100uf
Changed lines of the file:
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@@
   (symbol (lib_id "Device:C") (at 241.3 137.414 90) (unit 1)
     (in_bom yes) (on_board yes) (dnp no)
-    (property "Reference" "C7" (at 244.602 131.826 90)
+    (property "Reference" "C7" (at 241.554 130.048 90)
       (effects (font (size 1.27 1.27)))
     )
-    (property "Value" "C" (at 241.3 132.334 90)
+    (property "Value" "100uf" (at 241.3 132.334 90)
       (effects (font (size 1.27 1.27)))
     )

Commit message: Update
Changed lines of the file:
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@@
     (company "GERE")
   )
-  (junction (at 20.574 27.432) (diameter 0) (color 0 0 0 0)
-  )
   (junction (at 51.308 98.298) (diameter 0) (color 0 0 0 0)
   )
@@
   (junction (at 201.295 45.212) (diameter 0) (color 0 0 0 0)
   )
-  (junction (at 20.574 19.812) (diameter 0) (color 0 0 0 0)
+  (junction (at 20.828 19.812) (diameter 0) (color 0 0 0 0)
   )
   (junction (at 51.308 105.918) (diameter 0) (color 0 0 0 0)
@@
   (junction (at 207.645 32.512) (diameter 0) (color 0 0 0 0)
   )
+  (junction (at 20.828 27.432) (diameter 0) (color 0 0 0 0)
+  )
   (junction (at 181.61 45.847) (diameter 0) (color 0 0 0 0)
   )
@@
     (stroke (width 0) (type default))
   )
+  (wire (pts (xy 20.828 19.812) (xy 24.638 19.812))
+    (stroke (width 0) (type default))
+  )
   (wire (pts (xy 122.555 89.535) (xy 125.73 89.535))
     (stroke (width 0) (type default))
@@
     (stroke (width 0) (type default))
   )
+  (wire (pts (xy 20.828 29.718) (xy 20.828 27.432))
+    (stroke (width 0) (type default))
+  )
   (wire (pts (xy 104.14 41.91) (xy 110.49 41.91))
     (stroke (width 0) (type default))
@@
     (stroke (width 0) (type default))
   )
-  (wire (pts (xy 20.574 19.812) (xy 24.638 19.812))
-    (stroke (width 0) (type default))
-  )
   (wire (pts (xy 144.526 36.322) (xy 144.526 37.592))
     (stroke (width 0) (type default))
@@
     (stroke (width 0) (type default))
   )
-  (wire (pts (xy 20.574 27.432) (xy 20.574 29.21))
-    (stroke (width 0) (type default))
-  )
   (wire (pts (xy 44.704 81.28) (xy 44.704 81.534))
     (stroke (width 0) (type default))
@@
     (stroke (width 0) (type default))
   )
-  (wire (pts (xy 20.574 29.21) (xy 20.32 29.21))
+  (wire (pts (xy 20.828 27.432) (xy 20.828 19.812))
     (stroke (width 0) (type default))
   )
@@
     (stroke (width 0) (type default))
   )
-  (wire (pts (xy 16.764 19.812) (xy 20.574 19.812))
-    (stroke (width 0) (type default))
-  )
   (wire (pts (xy 122.555 109.855) (xy 125.73 109.855))
     (stroke (width 0) (type default))
@@
     (stroke (width 0) (type default))
   )
+  (wire (pts (xy 20.828 27.432) (xy 24.638 27.432))
+    (stroke (width 0) (type default))
+  )
   (wire (pts (xy 93.218 93.98) (xy 90.678 93.98))
     (stroke (width 0) (type default))
@@
     (stroke (width 0) (type default))
   )
-  (wire (pts (xy 20.574 27.432) (xy 24.638 27.432))
-    (stroke (width 0) (type default))
-  )
   (wire (pts (xy 181.61 32.512) (xy 181.61 38.227))
     (stroke (width 0) (type default))
@@
     (stroke (width 0) (type default))
   )
-  (wire (pts (xy 20.574 19.812) (xy 20.574 27.432))
-    (stroke (width 0) (type default))
-  )
   (wire (pts (xy 236.093 141.478) (xy 236.093 142.24))
     (stroke (width 0) (type default))
@@
     (stroke (width 0) (type default))
   )
-  (wire (pts (xy 16.256 27.432) (xy 20.574 27.432))
+  (wire (pts (xy 16.764 19.812) (xy 20.828 19.812))
     (stroke (width 0) (type default))
   )
@@
   )
   (wire (pts (xy 201.295 45.212) (xy 201.295 45.847))
+    (stroke (width 0) (type default))
+  )
+  (wire (pts (xy 16.256 27.432) (xy 20.828 27.432))
     (stroke (width 0) (type default))
   )
@@
         (path "/5740c1d8-40a5-48a4-b0ff-1fed8540b5f6"
           (reference "U3") (unit 1)
+        )
+      )
+    )
+  )
+  (symbol (lib_id "power:GND") (at 20.828 29.718 0) (unit 1)
+    (in_bom yes) (on_board yes) (dnp no) (fields_autoplaced)
+    (property "Reference" "#PWR026" (at 20.828 36.068 0)
+      (effects (font (size 1.27 1.27)) hide)
+    )
+    (property "Value" "GND" (at 20.828 34.29 0)
+      (effects (font (size 1.27 1.27)))
+    )
+    (property "Footprint" "" (at 20.828 29.718 0)
+      (effects (font (size 1.27 1.27)) hide)
+    )
+    (property "Datasheet" "" (at 20.828 29.718 0)
+      (effects (font (size 1.27 1.27)) hide)
+    )
+    (pin "1")
+    (instances
+      (project "Robot_PCB_(110x55mm)"
+        (path "/5740c1d8-40a5-48a4-b0ff-1fed8540b5f6"
+          (reference "#PWR026") (unit 1)
         )
       )
@@
         )
       )
-    )
-  )
-  (symbol (lib_id "power:GND") (at 20.32 29.21 0) (unit 1)
-    (in_bom yes) (on_board yes) (dnp no) (fields_autoplaced)
-    (property "Reference" "#PWR026" (at 20.32 35.56 0)
-      (effects (font (size 1.27 1.27)) hide)
-    )
-    (property "Value" "GND" (at 20.32 33.528 0)
-      (effects (font (size 1.27 1.27)))
-    )
-    (property "Footprint" "" (at 20.32 29.21 0)
-      (effects (font (size 1.27 1.27)) hide)
-    )
-    (property "Datasheet" "" (at 20.32 29.21 0)
-      (effects (font (size 1.27 1.27)) hide)
-    )
-    (pin "1")
-    (instances
-      (project "Robot_PCB_(110x55mm)"
-        (path "/5740c1d8-40a5-48a4-b0ff-1fed8540b5f6"
-          (reference "#PWR026") (unit 1)
-        )
-      )

Commit message: Update
Parts:
- H1, H2, H3, H4: footprint MountingHole:MountingHole_3.2mm_M3_ISO14580_Pad -> MountingHole:MountingHole_3.2mm_M3_DIN965_Pad
Changed lines of the file:
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@@
       (effects (font (size 1.27 1.27)) (justify left))
     )
-    (property "Footprint" "MountingHole:MountingHole_3.2mm_M3_ISO14580_Pad" (at 16.764 17.272 0)
+    (property "Footprint" "MountingHole:MountingHole_3.2mm_M3_DIN965_Pad" (at 16.764 17.272 0)
       (effects (font (size 1.27 1.27)) hide)
     )
@@
       (effects (font (size 1.27 1.27)) (justify left))
     )
-    (property "Footprint" "MountingHole:MountingHole_3.2mm_M3_ISO14580_Pad" (at 24.638 24.892 0)
+    (property "Footprint" "MountingHole:MountingHole_3.2mm_M3_DIN965_Pad" (at 24.638 24.892 0)
       (effects (font (size 1.27 1.27)) hide)
     )
@@
       (effects (font (size 1.27 1.27)) (justify left))
     )
-    (property "Footprint" "MountingHole:MountingHole_3.2mm_M3_ISO14580_Pad" (at 16.256 24.892 0)
+    (property "Footprint" "MountingHole:MountingHole_3.2mm_M3_DIN965_Pad" (at 16.256 24.892 0)
       (effects (font (size 1.27 1.27)) hide)
     )
@@
       (effects (font (size 1.27 1.27)) (justify left))
     )
-    (property "Footprint" "MountingHole:MountingHole_3.2mm_M3_ISO14580_Pad" (at 24.638 17.272 0)
-      (effects (font (size 1.27 1.27)) hide)
-    )
+    (property "Footprint" "MountingHole:MountingHole_3.2mm_M3_DIN965_Pad" (at 24.638 17.272 0)
+      (effects (font (size 1.27 1.27)) hide)
+    )

Commit message: Update
Parts:
- removed C2, C4: 100uf, Capacitor_SMD:C_0603_1608Metric, symbol Device:C
- removed C3: 10uf, Capacitor_SMD:C_0603_1608Metric, symbol Device:C
- added C2: 220uF_10V, Capacitor_THT:CP_Radial_D6.3mm_P2.50mm, symbol PCM_SL_Capacitors:220uF_10V
- C1: value 10uf -> 100nF; footprint Capacitor_SMD:C_0603_1608Metric -> Capacitor_SMD:C_0805_2012Metric_Pad1.18x1.45mm_HandSolder
- C5, C6: value C -> 100nF
Connections:
- net +5V: now also C2.1
- net GND: now also C2.2
Other:
- moved on the sheet: C1

Commit message: Update
Parts:
- renumbered MOTOR2 to MOTOR1, MOTOR1 to MOTOR2
Other:
- note added: "PCB PADs 3mm"
- moved on the sheet: H1, H2, H3, H4
Changed lines of the file:
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@@
   (junction (at 53.975 73.66) (diameter 0) (color 0 0 0 0)
   )
-  (junction (at 20.828 19.812) (diameter 0) (color 0 0 0 0)
+  (junction (at 27.432 35.306) (diameter 0) (color 0 0 0 0)
   )
   (junction (at 51.308 105.918) (diameter 0) (color 0 0 0 0)
@@
   (junction (at 53.975 81.28) (diameter 0) (color 0 0 0 0)
   )
-  (junction (at 20.828 27.432) (diameter 0) (color 0 0 0 0)
+  (junction (at 27.432 42.926) (diameter 0) (color 0 0 0 0)
   )
   (junction (at 235.712 137.16) (diameter 0) (color 0 0 0 0)
@@
     (stroke (width 0) (type default))
   )
-  (wire (pts (xy 20.828 19.812) (xy 24.638 19.812))
+  (wire (pts (xy 27.432 35.306) (xy 31.242 35.306))
     (stroke (width 0) (type default))
   )
@@
     (stroke (width 0) (type default))
   )
-  (wire (pts (xy 20.828 29.718) (xy 20.828 27.432))
+  (wire (pts (xy 27.432 45.212) (xy 27.432 42.926))
     (stroke (width 0) (type default))
   )
@@
     (stroke (width 0) (type default))
   )
-  (wire (pts (xy 20.828 27.432) (xy 20.828 19.812))
+  (wire (pts (xy 27.432 42.926) (xy 27.432 35.306))
     (stroke (width 0) (type default))
   )
@@
     (stroke (width 0) (type default))
   )
-  (wire (pts (xy 20.828 27.432) (xy 24.638 27.432))
+  (wire (pts (xy 27.432 42.926) (xy 31.242 42.926))
     (stroke (width 0) (type default))
   )
@@
     (stroke (width 0) (type default))
   )
-  (wire (pts (xy 16.764 19.812) (xy 20.828 19.812))
+  (wire (pts (xy 23.368 35.306) (xy 27.432 35.306))
     (stroke (width 0) (type default))
   )
@@
     (stroke (width 0) (type default))
   )
-  (wire (pts (xy 16.256 27.432) (xy 20.828 27.432))
+  (wire (pts (xy 22.86 42.926) (xy 27.432 42.926))
     (stroke (width 0) (type default))
   )
@@
     (fill (type none))
   )
+  (rectangle (start 14.986 23.368) (end 53.086 51.054)
+    (stroke (width 0) (type dash))
+    (fill (type none))
+  )
   (rectangle (start 15.494 59.69) (end 102.108 124.46)
     (stroke (width 0) (type dash))
@@
     (effects (font (size 1.27 1.27)) (justify left bottom))
   )
+  (text "PCB PADs 3mm " (at 16.51 26.162 0)
+    (effects (font (size 1.27 1.27)) (justify left bottom))
+  )
   (text "Power Button\n" (at 129.286 27.432 0)
     (effects (font (size 1.27 1.27)) (justify left bottom))
@@
   (symbol (lib_id "GERE_symbols:MOTOR ENC JST_06 (PH2.0) Horizontal") (at 43.434 118.618 0) (mirror y) (unit 1)
     (in_bom yes) (on_board yes) (dnp no) (fields_autoplaced)
-    (property "Reference" "MOTOR1" (at 39.624 100.33 0)
+    (property "Reference" "MOTOR2" (at 39.624 100.33 0)
       (effects (font (size 1.27 1.27)))
     )
@@
       (project "Robot_PCB_(110x55mm)"
         (path "/5740c1d8-40a5-48a4-b0ff-1fed8540b5f6"
-          (reference "MOTOR1") (unit 1)
+          (reference "MOTOR2") (unit 1)
         )
       )
@@
     )
   )
-  (symbol (lib_id "Mechanical:MountingHole_Pad") (at 16.764 17.272 0) (unit 1)
-    (in_bom yes) (on_board yes) (dnp no)
-    (property "Reference" "H2" (at 20.066 14.732 0)
-      (effects (font (size 1.27 1.27)) (justify left))
-    )
-    (property "Value" "MountingHole_Pad" (at 20.066 17.272 0)
-      (effects (font (size 1.27 1.27)) (justify left))
-    )
-    (property "Footprint" "MountingHole:MountingHole_3.2mm_M3_DIN965_Pad" (at 16.764 17.272 0)
-      (effects (font (size 1.27 1.27)) hide)
-    )
-    (property "Datasheet" "~" (at 16.764 17.272 0)
+  (symbol (lib_id "Mechanical:MountingHole_Pad") (at 23.368 32.766 0) (unit 1)
+    (in_bom yes) (on_board yes) (dnp no)
+    (property "Reference" "H2" (at 26.67 30.226 0)
+      (effects (font (size 1.27 1.27)) (justify left))
+    )
+    (property "Value" "MountingHole_Pad" (at 35.052 33.02 0)
+      (effects (font (size 1.27 1.27)) (justify left))
+    )
+    (property "Footprint" "MountingHole:MountingHole_3.2mm_M3_DIN965_Pad" (at 23.368 32.766 0)
+      (effects (font (size 1.27 1.27)) hide)
+    )
+    (property "Datasheet" "~" (at 23.368 32.766 0)
       (effects (font (size 1.27 1.27)) hide)
     )
@@
     )
   )
-  (symbol (lib_id "power:GND") (at 20.828 29.718 0) (unit 1)
-    (in_bom yes) (on_board yes) (dnp no) (fields_autoplaced)
-    (property "Reference" "#PWR026" (at 20.828 36.068 0)
-      (effects (font (size 1.27 1.27)) hide)
-    )
-    (property "Value" "GND" (at 20.828 34.29 0)
-      (effects (font (size 1.27 1.27)))
-    )
-    (property "Footprint" "" (at 20.828 29.718 0)
-      (effects (font (size 1.27 1.27)) hide)
-    )
-    (property "Datasheet" "" (at 20.828 29.718 0)
+  (symbol (lib_id "power:GND") (at 27.432 45.212 0) (unit 1)
+    (in_bom yes) (on_board yes) (dnp no) (fields_autoplaced)
+    (property "Reference" "#PWR026" (at 27.432 51.562 0)
+      (effects (font (size 1.27 1.27)) hide)
+    )
+    (property "Value" "GND" (at 27.432 49.784 0)
+      (effects (font (size 1.27 1.27)))
+    )
+    (property "Footprint" "" (at 27.432 45.212 0)
+      (effects (font (size 1.27 1.27)) hide)
+    )
+    (property "Datasheet" "" (at 27.432 45.212 0)
       (effects (font (size 1.27 1.27)) hide)
     )
@@
     )
   )
-  (symbol (lib_id "Mechanical:MountingHole_Pad") (at 24.638 24.892 0) (unit 1)
-    (in_bom yes) (on_board yes) (dnp no)
-    (property "Reference" "H4" (at 27.686 22.352 0)
-      (effects (font (size 1.27 1.27)) (justify left))
-    )
-    (property "Value" "MountingHole_Pad" (at 27.686 24.892 0)
-      (effects (font (size 1.27 1.27)) (justify left))
-    )
-    (property "Footprint" "MountingHole:MountingHole_3.2mm_M3_DIN965_Pad" (at 24.638 24.892 0)
-      (effects (font (size 1.27 1.27)) hide)
-    )
-    (property "Datasheet" "~" (at 24.638 24.892 0)
+  (symbol (lib_id "Mechanical:MountingHole_Pad") (at 31.242 40.386 0) (unit 1)
+    (in_bom yes) (on_board yes) (dnp no)
+    (property "Reference" "H4" (at 34.29 37.846 0)
+      (effects (font (size 1.27 1.27)) (justify left))
+    )
+    (property "Value" "MountingHole_Pad" (at 34.29 43.688 0)
+      (effects (font (size 1.27 1.27)) (justify left))
+    )
+    (property "Footprint" "MountingHole:MountingHole_3.2mm_M3_DIN965_Pad" (at 31.242 40.386 0)
+      (effects (font (size 1.27 1.27)) hide)
+    )
+    (property "Datasheet" "~" (at 31.242 40.386 0)
       (effects (font (size 1.27 1.27)) hide)
     )
@@
   (symbol (lib_id "GERE_symbols:MOTOR ENC JST_06 (PH2.0) Horizontal") (at 44.704 94.234 0) (mirror y) (unit 1)
     (in_bom yes) (on_board yes) (dnp no) (fields_autoplaced)
-    (property "Reference" "MOTOR2" (at 40.894 74.93 0)
+    (property "Reference" "MOTOR1" (at 40.894 74.93 0)
       (effects (font (size 1.27 1.27)))
     )
@@
       (project "Robot_PCB_(110x55mm)"
         (path "/5740c1d8-40a5-48a4-b0ff-1fed8540b5f6"
-          (reference "MOTOR2") (unit 1)
+          (reference "MOTOR1") (unit 1)
         )
       )
@@
     )
   )
-  (symbol (lib_id "Mechanical:MountingHole_Pad") (at 16.256 24.892 0) (unit 1)
-    (in_bom yes) (on_board yes) (dnp no)
-    (property "Reference" "H1" (at 18.796 22.352 0)
-      (effects (font (size 1.27 1.27)) (justify left))
-    )
-    (property "Value" "MountingHole_Pad" (at 18.796 24.892 0)
-      (effects (font (size 1.27 1.27)) (justify left))
-    )
-    (property "Footprint" "MountingHole:MountingHole_3.2mm_M3_DIN965_Pad" (at 16.256 24.892 0)
-      (effects (font (size 1.27 1.27)) hide)
-    )
-    (property "Datasheet" "~" (at 16.256 24.892 0)
+  (symbol (lib_id "Mechanical:MountingHole_Pad") (at 22.86 40.386 0) (unit 1)
+    (in_bom yes) (on_board yes) (dnp no)
+    (property "Reference" "H1" (at 25.4 37.846 0)
+      (effects (font (size 1.27 1.27)) (justify left))
+    )
+    (property "Value" "MountingHole_Pad" (at 34.29 41.656 0)
+      (effects (font (size 1.27 1.27)) (justify left))
+    )
+    (property "Footprint" "MountingHole:MountingHole_3.2mm_M3_DIN965_Pad" (at 22.86 40.386 0)
+      (effects (font (size 1.27 1.27)) hide)
+    )
+    (property "Datasheet" "~" (at 22.86 40.386 0)
       (effects (font (size 1.27 1.27)) hide)
     )
@@
     )
   )
-  (symbol (lib_id "Mechanical:MountingHole_Pad") (at 24.638 17.272 0) (unit 1)
-    (in_bom yes) (on_board yes) (dnp no)
-    (property "Reference" "H3" (at 27.686 14.732 0)
-      (effects (font (size 1.27 1.27)) (justify left))
-    )
-    (property "Value" "MountingHole_Pad" (at 27.686 17.272 0)
-      (effects (font (size 1.27 1.27)) (justify left))
-    )
-    (property "Footprint" "MountingHole:MountingHole_3.2mm_M3_DIN965_Pad" (at 24.638 17.272 0)
-      (effects (font (size 1.27 1.27)) hide)
-    )
-    (property "Datasheet" "~" (at 24.638 17.272 0)
-      (effects (font (size 1.27 1.27)) hide)
-    )
+  (symbol (lib_id "Mechanical:MountingHole_Pad") (at 31.242 32.766 0) (unit 1)
+    (in_bom yes) (on_board yes) (dnp no)
+    (property "Reference" "H3" (at 34.29 30.226 0)
+      (effects (font (size 1.27 1.27)) (justify left))
+    )
+    (property "Value" "MountingHole_Pad" (at 35.052 35.052 0)
+      (effects (font (size 1.27 1.27)) (justify left))
+    )
+    (property "Footprint" "MountingHole:MountingHole_3.2mm_M3_DIN965_Pad" (at 31.242 32.766 0)
+      (effects (font (size 1.27 1.27)) hide)
+    )
+    (property "Datasheet" "~" (at 31.242 32.766 0)
+      (effects (font (size 1.27 1.27)) hide)
+    )
