File: Robot_PCB_(110x55mm).kicad_sch (KiCad schematic)
At the start: 19 parts, among them U1 L293, U2 SW_DPDT_XLX, U3 AMS1117-5.0, U5 MFRC522 37.5x25mm

Commit message: Update
Connections:
- net +BATT: no longer U1.8 (VCC2)
- net VCC: now also U1.8 (VCC2)
Other:
- moved on the sheet: C1, C2, U3

Commit message: Update
Parts:
- added BZ1: Buzzer, Buzzer_Beeper:Buzzer_12x9.5RM7.6, symbol Device:Buzzer
- added Q1: J3, Package_TO_SOT_SMD:SOT-23_Handsoldering, symbol Transistor_BJT:MMBT3906
- added R1: 1000, Resistor_SMD:R_0805_2012Metric_Pad1.20x1.40mm_HandSolder, symbol Device:R
- added R2: 330, Resistor_SMD:R_0805_2012Metric_Pad1.20x1.40mm_HandSolder, symbol Device:R
- added R3: 680, Resistor_SMD:R_0805_2012Metric_Pad1.20x1.40mm_HandSolder, symbol Device:R
- SW1: renamed from U2; value SW_DPDT_XLX -> Switch; footprint GERE_footprints:SW_DPDT_XLX -> GERE_footprints:Push Button Switch 7mm
Connections:
- net +5V: now also Q1.3 (C)
- net Echo: now also R2.2, R3.1; no longer HC-SR04.2
- net GND: now also BZ1.2 (+), R3.2
- net BUZZER: now reaches A1.14 (D22/SCL)
- net BUZZER: now also R1.2
- new net: HC-SR04.2, R2.1
- new net: Q1.1 (B), R1.1
- new net: BZ1.1 (-), Q1.2 (E)
- no-connect marks 10 -> 9
Other:
- note added: "Buzzer"
- moved on the sheet: HC-SR04

Commit message: Update
Parts:
- removed HC-SR04: PINHD_1x4_Female, Connector_PinSocket_2.54mm:PinSocket_1x04_P2.54mm_Vertical, symbol PCM_SL_Pin_Headers:PINHD_1x4_Female
- added J1: HC-SR04, GERE_footprints:HC-SR04, symbol GERE_symbols:HC-SR04(Sonar)
- renumbered C2 to C1, C1 to C2, C5 to C3, C6 to C4, C7 to C5, U3 to U2
Connections:
- net +5V: now also J1.4 (Vcc)
- net GND: now also J1.1 (GND)
- net Trig: now also J1.3 (Echo)
- net at R2.1: now also J1.2 (Trig)
Changed lines of the file:
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@@
   (junction (at 248.92 76.2) (diameter 0) (color 0 0 0 0)
-  )
-  (junction (at 257.81 76.2) (diameter 0) (color 0 0 0 0)
   )
   (no_connect (at 175.26 119.38))
@@
     (stroke (width 0) (type default))
   )
+  (wire (pts (xy 257.81 76.2) (xy 259.08 76.2))
+    (stroke (width 0) (type default))
+  )
   (wire (pts (xy 248.92 46.99) (xy 247.65 46.99))
     (stroke (width 0) (type default))
@@
     (stroke (width 0) (type default))
   )
-  (wire (pts (xy 257.81 76.2) (xy 259.08 76.2))
-    (stroke (width 0) (type default))
-  )
   (wire (pts (xy 261.62 40.64) (xy 259.08 40.64))
     (stroke (width 0) (type default))
@@
   )
   (wire (pts (xy 175.26 88.9) (xy 177.8 88.9))
-    (stroke (width 0) (type default))
-  )
-  (wire (pts (xy 256.54 76.2) (xy 257.81 76.2))
     (stroke (width 0) (type default))
   )
@@
   (symbol (lib_id "Device:C") (at 190.5 38.1 0) (mirror x) (unit 1)
     (in_bom yes) (on_board yes) (dnp no)
-    (property "Reference" "C1" (at 186.69 36.83 0)
+    (property "Reference" "C2" (at 186.69 36.83 0)
       (effects (font (size 1.27 1.27)) (justify right))
     )
@@
       (project "Robot_PCB_(110x55mm)"
         (path "/5740c1d8-40a5-48a4-b0ff-1fed8540b5f6"
-          (reference "C1") (unit 1)
+          (reference "C2") (unit 1)
         )
       )
@@
   )
   (symbol (lib_id "power:GND") (at 248.92 46.99 90) (unit 1)
-    (in_bom yes) (on_board yes) (dnp no) (fields_autoplaced)
+    (in_bom yes) (on_board yes) (dnp no)
     (property "Reference" "#PWR033" (at 255.27 46.99 0)
       (effects (font (size 1.27 1.27)) hide)
     )
-    (property "Value" "GND" (at 252.73 46.99 90)
+    (property "Value" "GND" (at 250.19 49.53 90)
       (effects (font (size 1.27 1.27)) (justify right))
     )
@@
   (symbol (lib_id "Device:C") (at 254 76.2 90) (unit 1)
     (in_bom yes) (on_board yes) (dnp no)
-    (property "Reference" "C7" (at 254.254 68.834 90)
+    (property "Reference" "C5" (at 254.254 68.834 90)
       (effects (font (size 1.27 1.27)))
     )
@@
       (project "Robot_PCB_(110x55mm)"
         (path "/5740c1d8-40a5-48a4-b0ff-1fed8540b5f6"
-          (reference "C7") (unit 1)
+          (reference "C5") (unit 1)
         )
       )
@@
       (effects (font (size 1.27 1.27)) hide)
     )
-    (property "Value" "GND" (at 261.62 29.21 0)
+    (property "Value" "GND" (at 256.54 27.94 0)
       (effects (font (size 1.27 1.27)) (justify right))
     )
@@
   (symbol (lib_id "Regulator_Linear:AMS1117-5.0") (at 200.66 33.02 0) (unit 1)
     (in_bom yes) (on_board yes) (dnp no) (fields_autoplaced)
-    (property "Reference" "U3" (at 200.66 26.67 0)
+    (property "Reference" "U2" (at 200.66 26.67 0)
       (effects (font (size 1.27 1.27)))
     )
@@
       (project "Robot_PCB_(110x55mm)"
         (path "/5740c1d8-40a5-48a4-b0ff-1fed8540b5f6"
-          (reference "U3") (unit 1)
+          (reference "U2") (unit 1)
         )
       )
@@
   )
   (symbol (lib_id "power:VCC") (at 73.66 76.2 0) (unit 1)
-    (in_bom yes) (on_board yes) (dnp no) (fields_autoplaced)
+    (in_bom yes) (on_board yes) (dnp no)
     (property "Reference" "#PWR06" (at 73.66 80.01 0)
       (effects (font (size 1.27 1.27)) hide)
     )
-    (property "Value" "VCC" (at 73.66 71.12 0)
+    (property "Value" "VCC" (at 71.12 72.39 0)
       (effects (font (size 1.27 1.27)))
     )
@@
       (effects (font (size 1.27 1.27)) hide)
     )
-    (property "Value" "+5V" (at 264.16 43.18 0)
+    (property "Value" "+5V" (at 260.35 44.45 0)
       (effects (font (size 1.27 1.27)) (justify left))
     )
@@
         (path "/5740c1d8-40a5-48a4-b0ff-1fed8540b5f6"
           (reference "#PWR017") (unit 1)
+        )
+      )
+    )
+  )
+  (symbol (lib_id "GERE_symbols:HC-SR04(Sonar)") (at 264.16 40.64 0) (unit 1)
+    (in_bom yes) (on_board yes) (dnp no)
+    (property "Reference" "J1" (at 265.43 27.94 0)
+      (effects (font (size 1.27 1.27)) (justify left))
+    )
+    (property "Value" "HC-SR04" (at 261.62 45.72 0)
+      (effects (font (size 1.27 1.27)) (justify left))
+    )
+    (property "Footprint" "GERE_footprints:HC-SR04" (at 264.16 40.64 0)
+      (effects (font (size 1.27 1.27)) hide)
+    )
+    (property "Datasheet" "" (at 264.16 40.64 0)
+      (effects (font (size 1.27 1.27)) hide)
+    )
+    (pin "1")
+    (pin "2")
+    (pin "3")
+    (pin "4")
+    (instances
+      (project "Robot_PCB_(110x55mm)"
+        (path "/5740c1d8-40a5-48a4-b0ff-1fed8540b5f6"
+          (reference "J1") (unit 1)
         )
       )
@@
   (symbol (lib_id "PCM_SL_Capacitors:220uF_10V") (at 210.82 38.1 270) (unit 1)
     (in_bom yes) (on_board yes) (dnp no) (fields_autoplaced)
-    (property "Reference" "C2" (at 214.122 36.83 90)
+    (property "Reference" "C1" (at 214.122 36.83 90)
       (effects (font (size 1.27 1.27)) (justify left))
     )
@@
       (project "Robot_PCB_(110x55mm)"
         (path "/5740c1d8-40a5-48a4-b0ff-1fed8540b5f6"
-          (reference "C2") (unit 1)
+          (reference "C1") (unit 1)
         )
       )
@@
   (symbol (lib_id "Device:C") (at 50.8 114.3 0) (mirror x) (unit 1)
     (in_bom yes) (on_board yes) (dnp no) (fields_autoplaced)
-    (property "Reference" "C5" (at 54.102 115.57 0)
+    (property "Reference" "C3" (at 54.102 115.57 0)
       (effects (font (size 1.27 1.27)) (justify left))
     )
@@
       (project "Robot_PCB_(110x55mm)"
         (path "/5740c1d8-40a5-48a4-b0ff-1fed8540b5f6"
-          (reference "C5") (unit 1)
+          (reference "C3") (unit 1)
         )
       )
@@
   (symbol (lib_id "Device:C") (at 49.53 88.9 0) (mirror x) (unit 1)
     (in_bom yes) (on_board yes) (dnp no) (fields_autoplaced)
-    (property "Reference" "C6" (at 52.705 90.17 0)
+    (property "Reference" "C4" (at 52.705 90.17 0)
       (effects (font (size 1.27 1.27)) (justify left))
     )
@@
       (project "Robot_PCB_(110x55mm)"
         (path "/5740c1d8-40a5-48a4-b0ff-1fed8540b5f6"
-          (reference "C6") (unit 1)
+          (reference "C4") (unit 1)
         )
       )
@@
   (symbol (lib_id "Driver_Motor:L293") (at 76.2 104.14 0) (mirror y) (unit 1)
     (in_bom yes) (on_board yes) (dnp no)
-    (property "Reference" "U1" (at 71.4659 76.2 0)
-      (effects (font (size 1.27 1.27)) (justify left))
-    )
-    (property "Value" "L293" (at 71.4659 78.74 0)
+    (property "Reference" "U1" (at 68.58 74.93 0)
+      (effects (font (size 1.27 1.27)) (justify left))
+    )
+    (property "Value" "L293" (at 68.58 77.47 0)
       (effects (font (size 1.27 1.27)) (justify left))
     )
@@
     )
   )
-  (symbol (lib_id "PCM_SL_Pin_Headers:PINHD_1x4_Female") (at 265.43 36.83 0) (unit 1)
-    (in_bom yes) (on_board yes) (dnp no)
-    (property "Reference" "HC-SR04" (at 268.478 41.656 90)
-      (effects (font (size 1.27 1.27)) (justify left))
-    )
-    (property "Value" "PINHD_1x4_Female" (at 267.97 38.1 0)
-      (effects (font (size 1.27 1.27)) (justify left) hide)
-    )
-    (property "Footprint" "Connector_PinSocket_2.54mm:PinSocket_1x04_P2.54mm_Vertical" (at 267.97 24.13 0)
-      (effects (font (size 1.27 1.27)) hide)
-    )
-    (property "Datasheet" "" (at 265.43 26.67 0)
-      (effects (font (size 1.27 1.27)) hide)
-    )
-    (property "Campo4" "" (at 265.43 36.83 90)
-      (effects (font (size 1.27 1.27)) hide)
-    )
-    (pin "1")
-    (pin "2")
-    (pin "3")
-    (pin "4")
-    (instances
-      (project "Robot_PCB_(110x55mm)"
-        (path "/5740c1d8-40a5-48a4-b0ff-1fed8540b5f6"
-          (reference "HC-SR04") (unit 1)
-        )
-      )
-    )
-  )
   (symbol (lib_id "Device:R") (at 247.65 43.18 0) (unit 1)
     (in_bom yes) (on_board yes) (dnp no)
@@
   (symbol (lib_id "PCM_SL_Connectors:JST_02") (at 93.98 40.64 180) (unit 1)
     (in_bom yes) (on_board yes) (dnp no)
-    (property "Reference" "BAT1" (at 88.646 41.91 0)
+    (property "Reference" "BAT1" (at 88.9 39.37 0)
       (effects (font (size 1.27 1.27)))
     )
     (property "Value" "JST_02" (at 88.138 39.878 0)
-      (effects (font (size 1.27 1.27)))
+      (effects (font (size 1.27 1.27)) hide)
     )
     (property "Footprint" "Connector_JST:JST_EH_B2B-EH-A_1x02_P2.50mm_Vertical" (at 93.98 46.99 0)

Commit message: Update
Parts:
- removed BZ1: Buzzer, Buzzer_Beeper:Buzzer_12x9.5RM7.6, symbol Device:Buzzer
- removed Q1: J3, Package_TO_SOT_SMD:SOT-23_Handsoldering, symbol Transistor_BJT:MMBT3906
- added D1: LED, LED_THT:LED_D3.0mm_Clear, symbol Device:LED
- R1: value 1000 -> ~; Campo4 102 -> (none)
Connections:
- net GND: now also D1.1 (K)
- net at R1.1: now also D1.2 (A)
- net BUZZER renamed LED
Other:
- note added: "LED"
- note removed: "Buzzer"
- moved on the sheet: R1
Changed lines of the file:
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@@
-    (stroke (width 0) (type default))
-  )
-  (wire (pts (xy 64.77 172.72) (xy 64.77 173.99))
-    (stroke (width 0) (type default))
-  )
-  (wire (pts (xy 64.77 184.15) (xy 80.01 184.15))
     (stroke (width 0) (type default))
   )
@@
     (stroke (width 0) (type default))
   )
-  (wire (pts (xy 77.47 177.8) (xy 77.47 179.07))
-    (stroke (width 0) (type default))
-  )
   (wire (pts (xy 200.66 44.45) (xy 210.82 44.45))
     (stroke (width 0) (type default))
@@
     (stroke (width 0) (type default))
   )
+  (wire (pts (xy 63.5 175.26) (xy 66.04 175.26))
+    (stroke (width 0) (type default))
+  )
   (wire (pts (xy 127 93.98) (xy 130.81 93.98))
     (stroke (width 0) (type default))
   )
-  (wire (pts (xy 46.99 179.07) (xy 48.26 179.07))
+  (wire (pts (xy 45.72 175.26) (xy 46.99 175.26))
     (stroke (width 0) (type default))
   )
@@
     (stroke (width 0) (type default))
   )
-  (wire (pts (xy 55.88 179.07) (xy 57.15 179.07))
-    (stroke (width 0) (type default))
-  )
   (wire (pts (xy 208.28 33.02) (xy 210.82 33.02))
     (stroke (width 0) (type default))
@@
     (stroke (width 0) (type default))
   )
-  (wire (pts (xy 77.47 179.07) (xy 80.01 179.07))
-    (stroke (width 0) (type default))
-  )
   (wire (pts (xy 91.44 93.98) (xy 88.9 93.98))
     (stroke (width 0) (type default))
@@
   )
   (wire (pts (xy 49.53 93.98) (xy 49.53 92.71))
+    (stroke (width 0) (type default))
+  )
+  (wire (pts (xy 55.88 175.26) (xy 54.61 175.26))
     (stroke (width 0) (type default))
   )
@@
     (effects (font (size 1.27 1.27)) (justify left bottom))
   )
-  (text "Buzzer" (at 30.48 165.1 0)
+  (text "LED" (at 30.48 165.1 0)
     (effects (font (size 1.27 1.27)) (justify left bottom))
   )
@@
     )
   )
-  (global_label "BUZZER" (shape input) (at 46.99 179.07 180) (fields_autoplaced)
-    (effects (font (size 1.27 1.27)) (justify right))
-    (property "Intersheetrefs" "${INTERSHEET_REFS}" (at 36.5663 179.07 0)
-      (effects (font (size 1.27 1.27)) (justify right) hide)
-    )
-  )
-  (global_label "BUZZER" (shape input) (at 127 121.92 180) (fields_autoplaced)
-    (effects (font (size 1.27 1.27)) (justify right))
-    (property "Intersheetrefs" "${INTERSHEET_REFS}" (at 116.5763 121.92 0)
+  (global_label "LED" (shape input) (at 45.72 175.26 180) (fields_autoplaced)
+    (effects (font (size 1.27 1.27)) (justify right))
+    (property "Intersheetrefs" "${INTERSHEET_REFS}" (at 39.2877 175.26 0)
+      (effects (font (size 1.27 1.27)) (justify right) hide)
+    )
+  )
+  (global_label "LED" (shape input) (at 127 121.92 180) (fields_autoplaced)
+    (effects (font (size 1.27 1.27)) (justify right))
+    (property "Intersheetrefs" "${INTERSHEET_REFS}" (at 120.5677 121.92 0)
       (effects (font (size 1.27 1.27)) (justify right) hide)
     )
@@
         (path "/5740c1d8-40a5-48a4-b0ff-1fed8540b5f6"
           (reference "#PWR030") (unit 1)
-        )
-      )
-    )
-  )
-  (symbol (lib_id "power:+5V") (at 64.77 172.72 0) (unit 1)
-    (in_bom yes) (on_board yes) (dnp no) (fields_autoplaced)
-    (property "Reference" "#PWR031" (at 64.77 176.53 0)
-      (effects (font (size 1.27 1.27)) hide)
-    )
-    (property "Value" "+5V" (at 64.77 167.64 0)
-      (effects (font (size 1.27 1.27)))
-    )
-    (property "Footprint" "" (at 64.77 172.72 0)
-      (effects (font (size 1.27 1.27)) hide)
-    )
-    (property "Datasheet" "" (at 64.77 172.72 0)
-      (effects (font (size 1.27 1.27)) hide)
-    )
-    (pin "1")
-    (instances
-      (project "Robot_PCB_(110x55mm)"
-        (path "/5740c1d8-40a5-48a4-b0ff-1fed8540b5f6"
-          (reference "#PWR031") (unit 1)
         )
       )
@@
     )
   )
+  (symbol (lib_id "power:GND") (at 66.04 175.26 90) (unit 1)
+    (in_bom yes) (on_board yes) (dnp no)
+    (property "Reference" "#PWR027" (at 72.39 175.26 0)
+      (effects (font (size 1.27 1.27)) hide)
+    )
+    (property "Value" "GND" (at 68.58 177.8 90)
+      (effects (font (size 1.27 1.27)) (justify right))
+    )
+    (property "Footprint" "" (at 66.04 175.26 0)
+      (effects (font (size 1.27 1.27)) hide)
+    )
+    (property "Datasheet" "" (at 66.04 175.26 0)
+      (effects (font (size 1.27 1.27)) hide)
+    )
+    (pin "1")
+    (instances
+      (project "Robot_PCB_(110x55mm)"
+        (path "/5740c1d8-40a5-48a4-b0ff-1fed8540b5f6"
+          (reference "#PWR027") (unit 1)
+        )
+      )
+    )
+  )
   (symbol (lib_id "Device:R") (at 247.65 34.29 0) (unit 1)
     (in_bom yes) (on_board yes) (dnp no)
@@
     )
   )
-  (symbol (lib_id "Device:R") (at 52.07 179.07 270) (unit 1)
-    (in_bom yes) (on_board yes) (dnp no)
-    (property "Reference" "R1" (at 52.07 172.72 90)
-      (effects (font (size 1.27 1.27)))
-    )
-    (property "Value" "1000" (at 52.07 175.26 90)
-      (effects (font (size 1.27 1.27)))
-    )
-    (property "Footprint" "Resistor_SMD:R_0805_2012Metric_Pad1.20x1.40mm_HandSolder" (at 52.07 177.292 90)
-      (effects (font (size 1.27 1.27)) hide)
-    )
-    (property "Datasheet" "~" (at 52.07 179.07 0)
-      (effects (font (size 1.27 1.27)) hide)
-    )
-    (property "Campo4" "102" (at 52.07 181.61 90)
-      (effects (font (size 1.27 1.27)))
+  (symbol (lib_id "Device:R") (at 50.8 175.26 270) (unit 1)
+    (in_bom yes) (on_board yes) (dnp no)
+    (property "Reference" "R1" (at 50.8 168.91 90)
+      (effects (font (size 1.27 1.27)))
+    )
+    (property "Value" "~" (at 50.8 171.45 90)
+      (effects (font (size 1.27 1.27)))
+    )
+    (property "Footprint" "Resistor_SMD:R_0805_2012Metric_Pad1.20x1.40mm_HandSolder" (at 50.8 173.482 90)
+      (effects (font (size 1.27 1.27)) hide)
+    )
+    (property "Datasheet" "~" (at 50.8 175.26 0)
+      (effects (font (size 1.27 1.27)) hide)
     )
     (pin "1")
@@
         (path "/5740c1d8-40a5-48a4-b0ff-1fed8540b5f6"
           (reference "#PWR04") (unit 1)
-        )
-      )
-    )
-  )
-  (symbol (lib_id "power:GND") (at 77.47 177.8 0) (mirror x) (unit 1)
-    (in_bom yes) (on_board yes) (dnp no)
-    (property "Reference" "#PWR027" (at 77.47 171.45 0)
-      (effects (font (size 1.27 1.27)) hide)
-    )
-    (property "Value" "GND" (at 77.47 172.72 0)
-      (effects (font (size 1.27 1.27)))
-    )
-    (property "Footprint" "" (at 77.47 177.8 0)
-      (effects (font (size 1.27 1.27)) hide)
-    )
-    (property "Datasheet" "" (at 77.47 177.8 0)
-      (effects (font (size 1.27 1.27)) hide)
-    )
-    (pin "1")
-    (instances
-      (project "Robot_PCB_(110x55mm)"
-        (path "/5740c1d8-40a5-48a4-b0ff-1fed8540b5f6"
-          (reference "#PWR027") (unit 1)
         )
       )
@@
     )
   )
-  (symbol (lib_id "Transistor_BJT:MMBT3906") (at 62.23 179.07 0) (unit 1)
-    (in_bom yes) (on_board yes) (dnp no) (fields_autoplaced)
-    (property "Reference" "Q1" (at 67.31 177.8 0)
-      (effects (font (size 1.27 1.27)) (justify left))
-    )
-    (property "Value" "J3" (at 67.31 180.34 0)
-      (effects (font (size 1.27 1.27)) (justify left))
-    )
-    (property "Footprint" "Package_TO_SOT_SMD:SOT-23_Handsoldering" (at 67.31 180.975 0)
-      (effects (font (size 1.27 1.27) italic) (justify left) hide)
-    )
-    (property "Datasheet" "https://www.onsemi.com/pdf/datasheet/pzt3906-d.pdf" (at 62.23 179.07 0)
-      (effects (font (size 1.27 1.27)) (justify left) hide)
-    )
-    (pin "1")
-    (pin "2")
-    (pin "3")
-    (instances
-      (project "Robot_PCB_(110x55mm)"
-        (path "/5740c1d8-40a5-48a4-b0ff-1fed8540b5f6"
-          (reference "Q1") (unit 1)
-        )
-      )
-    )
-  )
   (symbol (lib_id "power:GND") (at 259.08 76.2 90) (unit 1)
     (in_bom yes) (on_board yes) (dnp no)
@@
         (path "/5740c1d8-40a5-48a4-b0ff-1fed8540b5f6"
           (reference "#PWR029") (unit 1)
+        )
+      )
+    )
+  )
+  (symbol (lib_id "Device:LED") (at 59.69 175.26 0) (mirror y) (unit 1)
+    (in_bom yes) (on_board yes) (dnp no)
+    (property "Reference" "D1" (at 61.2775 168.91 0)
+      (effects (font (size 1.27 1.27)))
+    )
+    (property "Value" "LED" (at 61.2775 171.45 0)
+      (effects (font (size 1.27 1.27)))
+    )
+    (property "Footprint" "LED_THT:LED_D3.0mm_Clear" (at 59.69 175.26 0)
+      (effects (font (size 1.27 1.27)) hide)
+    )
+    (property "Datasheet" "~" (at 59.69 175.26 0)
+      (effects (font (size 1.27 1.27)) hide)
+    )
+    (pin "1")
+    (pin "2")
+    (instances
+      (project "Robot_PCB_(110x55mm)"
+        (path "/5740c1d8-40a5-48a4-b0ff-1fed8540b5f6"
+          (reference "D1") (unit 1)
         )
       )
@@
         )
       )
-    )
-  )
-  (symbol (lib_id "Device:Buzzer") (at 82.55 181.61 0) (mirror x) (unit 1)
-    (in_bom yes) (on_board yes) (dnp no)
-    (property "Reference" "BZ1" (at 82.0351 185.42 90)
-      (effects (font (size 1.27 1.27)) (justify left) hide)
-    )
-    (property "Value" "Buzzer" (at 83.3051 176.53 0)
-      (effects (font (size 1.27 1.27)))
-    )
-    (property "Footprint" "Buzzer_Beeper:Buzzer_12x9.5RM7.6" (at 81.915 184.15 90)
-      (effects (font (size 1.27 1.27)) hide)
-    )
-    (property "Datasheet" "~" (at 81.915 184.15 90)
-      (effects (font (size 1.27 1.27)) hide)
-    )
-    (pin "1")
-    (pin "2")
-    (instances
-      (project "Robot_PCB_(110x55mm)"
-        (path "/5740c1d8-40a5-48a4-b0ff-1fed8540b5f6"
-          (reference "BZ1") (unit 1)
-        )
-      )

Commit message: Update
Parts:
- MOTOR1, MOTOR2: footprint Connector_JST:JST_PH_S6B-PH-K_1x06_P2.00mm_Horizontal -> GERE_footprints:Encoder Socket
Changed lines of the file:
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@@
       (effects (font (size 1.27 1.27)) hide)
     )
-    (property "Footprint" "Connector_JST:JST_PH_S6B-PH-K_1x06_P2.00mm_Horizontal" (at 13.97 95.25 0)
+    (property "Footprint" "GERE_footprints:Encoder Socket" (at 13.97 95.25 0)
       (effects (font (size 1.27 1.27)) hide)
     )
@@
       (effects (font (size 1.27 1.27)) hide)
     )
-    (property "Footprint" "Connector_JST:JST_PH_S6B-PH-K_1x06_P2.00mm_Horizontal" (at 13.97 69.85 0)
-      (effects (font (size 1.27 1.27)) hide)
-    )
+    (property "Footprint" "GERE_footprints:Encoder Socket" (at 13.97 69.85 0)
+      (effects (font (size 1.27 1.27)) hide)
+    )
